Commit message: ubuntu18

File: catkin_ws/src/mbot_description/urdf/mbot_with_laser.urdf (robot description, URDF)
Before this commit: robot mbot, 5 links, 4 joints
Links:
- added link laser_link; visual cylinder length=0.05 radius=0.05
Joints:
- added joint laser_joint: type fixed, parent base_link, child laser_link, origin xyz=0 0 0.105 rpy=0 0 0
